File: etc/schematics/Transmitter_ks0108_version.sch (EAGLE design)
At the start: 67 parts, among them IC1 ATMEGA328P, IC2 ATMEGA328P, IC3 74HC595N, Q1 16MHz, Q2 16MHz, T1 BC337, T2 BC337, U1 AMS1117_3.3

Commit message: Add files via upload
Parts:
- added C14: 100n, rcl:C-EU025-025X050
- added CONN17: (no value), con-lstb:MA03-1
- added D5: 1N5819, diode:1N5817-B
- added IC4: 7805T, linear:7805T
- added OK1: PC817, optocoupler:PC817
- added Q4: P_MOSFET, transistor-power:FDN360P
- added R27: 1k, rcl:R-US_0204/2V
- added R28, R31, R32: 220k, rcl:R-US_0204/7
- added R29, R35: 10k, rcl:R-US_0204/7
- added R33, R34: 220, rcl:R-US_0204/7
- added T3: BC337, transistor:BC337
Connections:
- new net N$38: OK1.EMIT, R3.1
- new net N$39: C14.2, CONN1.1, CONN1.2, Q4.S, R28.2, R29.2
- new net N$43: C14.1, Q4.G, R28.1, T3.C
- new net N$44: OK1.C, R27.2
- new net N$45: CONN17.1, R29.1
- new net N$47: C5.+, IC4.VI, Q4.D
- new net N$49: CONN2.2, R33.1
- new net N$50: CONN2.1, R34.1
- new net N$51: IC2.PC3(ADC3), R33.2
- new net N$52: IC2.PC2(ADC2), R34.2
- new net N$53: R31.1, R35.1, T3.B
- new net N$54: CONN17.2, D5.C, R35.2
- new net POW_LATCH: D5.A, IC2.PC0(ADC0)
- new net POW_OFF: CONN17.3, IC2.PC1(ADC1), R32.1
- net +5V: now also IC4.VO, OK1.A; no longer C5.+, CONN1.1, CONN1.2
- net GND: now also IC4.GND, R27.1, R31.2, R32.2, T3.E
- net N$1: now also OK1.COL; no longer R3.1
Other:
- note added: "220 ohms"
- note added: "Power switch (Slide type)"
- note added: "RC Transmitter Schematic by BUK7456 2020-2021"
- note added: "SWC_LOWERPOS"
- note added: "SWC_UPPERPOS"
- note added: "SWE"
- note added: "SWF"
- note added: "Soft power latch circuit is optional"
- note added: "The max voltage here should not exceed 4.7V, so the resistors in this voltage divider should be sized appropriately"
- note added: "V_IN"
- note added: "V_IN is 7-12V. VBATT and V_IN can be shorted together e.g. when using 2 series Li-ion cells."
- note removed: "5V IN"
- note removed: "RC Transmitter Schematic by BUK7456 2020"
- note removed: "SWC"
- note removed: "The max voltage here should not exceed 5V, so the resistors in this voltage divider should be sized appropriately"
- note removed: "upperPos lowerPos common"
- moved on the sheet: C1, C10, C11, C12, C13, C2, C3, C4, C5, C6, C7, C8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
